File: schematic/WirelessPalaControl.kicad_pcb (KiCad board)
At the start: 2 copper layers, 25.4 x 34.3 mm, 18 parts, among them J1 6P4C, J2 MCU UART, J3 WeMos_mini_Hat_Left, J4 WeMos_mini_Hat_Right, U1 SI8621

Commit message: Change R4 to 2K
Parts:
- R4: value 10K -> 2K
Other:
- board text added: "C1,C2: 100n D1,D3: Red Led D2: SS34 R1,R6: 1K R2,R7: 220 R3,R4,R8: 2K R5: 10K U1: Si8621"
- board text removed: "C1,C2: 100n D1,D3: Red Led D2: SS34 R1,R6: 1K R2,R7: 220 R3,R8: 2K R4,R5: 10K U1: Si8621"
Changed lines of the file:
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@@
 			)
 		)
-		(property "Value" "10K"
+		(property "Value" "2K"
 			(at 0 1.65 180)
 			(layer "F.Fab")
@@
 			)
 		)
-		(property "LCSC" "C17414"
+		(property "LCSC" "C17604"
 			(at 0 0 180)
 			(unlocked yes)
@@
 		)
 	)
-	(gr_text "C1,C2: 100n\nD1,D3: Red Led\nD2: SS34\nR1,R6: 1K\nR2,R7: 220\nR3,R8: 2K\nR4,R5: 10K\nU1: Si8621"
+	(gr_text "C1,C2: 100n\nD1,D3: Red Led\nD2: SS34\nR1,R6: 1K\nR2,R7: 220\nR3,R4,R8: 2K\nR5: 10K\nU1: Si8621"
 		(at 40.64 48.641 0)
 		(layer "B.SilkS")
